File: kicad/midi_io.sch (KiCad schematic (older format))
At the start: 10 parts, among them J1 MIDI Out, J2 MIDI In, J3 Conn_01x04, U1 6N138

Commit message: Change to 0804 SMD resistors
Parts:
- R1, R2, R3, R4, R5: footprint Resistor_THT:R_Axial_DIN0207_L6.3mm_D2.5mm_P7.62mm_Horizontal -> Resistor_SMD:R_0805_2012Metric_Pad1.15x1.40mm_HandSolder
Changed lines of the file:
@@
 F 0 "R1" V 5143 4450 50  0000 C CNN
 F 1 "220" V 5234 4450 50  0000 C CNN
-F 2 "Resistor_THT:R_Axial_DIN0207_L6.3mm_D2.5mm_P7.62mm_Horizontal" V 5280 4450 50  0001 C CNN
+F 2 "Resistor_SMD:R_0805_2012Metric_Pad1.15x1.40mm_HandSolder" V 5280 4450 50  0001 C CNN
 F 3 "~" H 5350 4450 50  0001 C CNN
 	1    5350 4450
@@
 F 0 "R2" V 4543 4450 50  0000 C CNN
 F 1 "220" V 4634 4450 50  0000 C CNN
-F 2 "Resistor_THT:R_Axial_DIN0207_L6.3mm_D2.5mm_P7.62mm_Horizontal" V 4680 4450 50  0001 C CNN
+F 2 "Resistor_SMD:R_0805_2012Metric_Pad1.15x1.40mm_HandSolder" V 4680 4450 50  0001 C CNN
 F 3 "~" H 4750 4450 50  0001 C CNN
 	1    4750 4450
@@
 F 0 "R5" H 6920 3396 50  0000 L CNN
 F 1 "4.7k" H 6920 3305 50  0000 L CNN
-F 2 "Resistor_THT:R_Axial_DIN0207_L6.3mm_D2.5mm_P7.62mm_Horizontal" V 6780 3350 50  0001 C CNN
+F 2 "Resistor_SMD:R_0805_2012Metric_Pad1.15x1.40mm_HandSolder" V 6780 3350 50  0001 C CNN
 F 3 "~" H 6850 3350 50  0001 C CNN
 	1    6850 3350
@@
 F 0 "R4" H 7170 2796 50  0000 L CNN
 F 1 "220" H 7170 2705 50  0000 L CNN
-F 2 "Resistor_THT:R_Axial_DIN0207_L6.3mm_D2.5mm_P7.62mm_Horizontal" V 7030 2750 50  0001 C CNN
+F 2 "Resistor_SMD:R_0805_2012Metric_Pad1.15x1.40mm_HandSolder" V 7030 2750 50  0001 C CNN
 F 3 "~" H 7100 2750 50  0001 C CNN
 	1    7100 2750
@@
 F 0 "R3" V 5193 2450 50  0000 C CNN
 F 1 "220" V 5284 2450 50  0000 C CNN
-F 2 "Resistor_THT:R_Axial_DIN0207_L6.3mm_D2.5mm_P7.62mm_Horizontal" V 5330 2450 50  0001 C CNN
+F 2 "Resistor_SMD:R_0805_2012Metric_Pad1.15x1.40mm_HandSolder" V 5330 2450 50  0001 C CNN
 F 3 "~" H 5400 2450 50  0001 C CNN
 	1    5400 2450
