File: kicad/midi_io.sch (KiCad schematic (older format))
At the start: 10 parts, among them J1 MIDI Out, J2 MIDI In, J3 Conn_01x04, U1 6N138

Commit message: Update with fixes from first prototype
Parts:
- D1: MPN (none) -> 1N4001-G
- J3: footprint Connector_PinHeader_2.54mm:PinHeader_1x04_P2.54mm_Vertical -> Connector_PinSocket_2.54mm:PinSocket_1x04_P2.54mm_Vertical
- U1: MPN (none) -> 6N138
Changed lines of the file:
@@
 F 5 "1" H 6500 2950 50  0001 C CNN "Spice_Model"
 F 6 "Y" H 6500 2950 50  0001 C CNN "Spice_Netlist_Enabled"
+F 7 "6N138" H 6500 2950 50  0001 C CNN "MPN"
 	1    6500 2950
 	1    0    0    -1
@@
 F 0 "J3" H 6930 4542 50  0000 L CNN
 F 1 "Conn_01x04" H 6930 4451 50  0000 L CNN
-F 2 "Connector_PinHeader_2.54mm:PinHeader_1x04_P2.54mm_Vertical" H 6850 4550 50  0001 C CNN
+F 2 "Connector_PinSocket_2.54mm:PinSocket_1x04_P2.54mm_Vertical" H 6850 4550 50  0001 C CNN
 F 3 "~" H 6850 4550 50  0001 C CNN
 F 4 "R" H 6850 4550 50  0001 C CNN "Spice_Primitive"
@@
 F 5 "1" H 5750 2850 50  0001 C CNN "Spice_Model"
 F 6 "Y" H 5750 2850 50  0001 C CNN "Spice_Netlist_Enabled"
+F 7 "1N4001-G" H 5750 2850 50  0001 C CNN "MPN"
 	1    5750 2850
 	0    1    1    0
