File: midi_io/midi_io.kicad_pcb (KiCad board)
At the start: 2 copper layers, 35.6 x 41.4 mm, 10 parts, among them J1 MIDI Out, J2 MIDI In, J3 Conn_01x04, U1 6N138

Commit message: Rename 5V silk to VCC
Other:
- board text added: "VCC"
- board text removed: "5V"
Changed lines of the file:
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@@
-(kicad_pcb (version 20171130) (host pcbnew "(5.1.5-0-10_14)")
+(kicad_pcb (version 20171130) (host pcbnew 5.1.5-52549c5~84~ubuntu18.04.1)
   (general
     (thickness 1.6)
@@
     (effects (font (size 0.9652 0.9652) (thickness 0.1524)) (justify right))
   )
-  (gr_text "5V\n" (at 162.433 106.68) (layer F.SilkS)
+  (gr_text "VCC\n" (at 162.433 106.68) (layer F.SilkS)
     (effects (font (size 0.9652 0.9652) (thickness 0.1524)) (justify right))
   )
